File: pcbTemas/pcbTemas.kicad_sch (KiCad schematic)
At the start: 1 part, among them U1 ESP32-WROOM-32D

Commit message: actualizacion pcb
Parts:
- removed U1: ESP32-WROOM-32D, RF_Module:ESP32-WROOM-32D, symbol RF_Module:ESP32-WROOM-32D
- added BIDIR, INPUT, OUTPUT: Conn_02x08_Odd_Even, Connector_PinHeader_2.54mm:PinHeader_2x08_P2.54mm_Horizontal, symbol Connector_Generic:Conn_02x08_Odd_Even
- added FLASH, RAM: Conn_01x06, Connector_PinHeader_2.54mm:PinHeader_1x06_P2.54mm_Horizontal, symbol Connector_Generic:Conn_01x06
- added J1: Conn_01x02, symbol Connector_Generic:Conn_01x02
- added Logic_analizer: Conn_02x05_Odd_Even, symbol Connector_Generic:Conn_02x05_Odd_Even
- added U1: 74LS157, symbol 74xx:74LS157
Connections:
- new net +3.3V: FLASH.1 (Pin_1), J1.1 (Pin_1), RAM.6 (Pin_6), U1.16 (VCC)
- new net CH1: Logic_analizer.1 (Pin_1)
- new net CH2: Logic_analizer.2 (Pin_2)
- new net CH3: Logic_analizer.3 (Pin_3)
- new net CH4: Logic_analizer.4 (Pin_4)
- new net CH5: Logic_analizer.5 (Pin_5)
- new net CH6: Logic_analizer.6 (Pin_6)
- new net CH7: Logic_analizer.7 (Pin_7)
- new net CH8: Logic_analizer.8 (Pin_8)
- new net CLK: Logic_analizer.9 (Pin_9)
- new net CS_FLASH: FLASH.2 (Pin_2), U1.2 (I0a)
- new net CS_RAM: RAM.1 (Pin_1), U1.3 (I1a)
- new net GND: FLASH.4 (Pin_4), J1.2 (Pin_2), Logic_analizer.10 (Pin_10), RAM.5 (Pin_5), U1.8 (GND)
- new net MISO: FLASH.3 (Pin_3), RAM.3 (Pin_3)
- new net MOSI: FLASH.6 (Pin_6), RAM.2 (Pin_2)
- new net SCLK: FLASH.5 (Pin_5), RAM.4 (Pin_4)
